Commit message: uptimized for more speed

File: install/robokpy_controller/share/robokpy_controller/urdf/ur5e_virtual_robotiq_85_gripper.urdf (robot description, URDF)
Before this commit: robot ur_robot, 23 links, 22 joints
Joints:
- removed joint tool0-tcp
- added joint robotiq_85_base_link-tcp: type fixed, parent robotiq_85_base_link, child tcp, origin xyz=0.104 0 0 rpy=0 1.5707963267948966 0
