Commit message: Fixing Motus CLI

File: mycobot_pi/install/mycobot_pi_motus/share/mycobot_pi_motus/urdf/mycobot_pi.urdf.xacro (robot description, xacro)
@@ -40,4 +40,9 @@
   </link>
   <link name="joint2">
+    <inertial>
+      <mass value="0.001"/>
+      <origin xyz="0 0 0" rpy="0 0 0"/>
+      <inertia ixx="0.0001" iyy="0.0001" izz="0.0001" ixy="0" ixz="0" iyz="0"/>
+    </inertial>
     <visual>
       <geometry>
@@ -54,4 +59,9 @@
   </link>
   <link name="joint3">
+    <inertial>
+      <mass value="0.001"/>
+      <origin xyz="0 0 0" rpy="0 0 0"/>
+      <inertia ixx="0.0001" iyy="0.0001" izz="0.0001" ixy="0" ixz="0" iyz="0"/>
+    </inertial>
     <visual>
       <geometry>
@@ -68,4 +78,9 @@
   </link>
   <link name="joint4">
+    <inertial>
+      <mass value="0.001"/>
+      <origin xyz="0 0 0" rpy="0 0 0"/>
+      <inertia ixx="0.0001" iyy="0.0001" izz="0.0001" ixy="0" ixz="0" iyz="0"/>
+    </inertial>
     <visual>
       <geometry>
@@ -84,4 +99,9 @@
   </link>
 <link name="joint5">
+    <inertial>
+      <mass value="0.001"/>
+      <origin xyz="0 0 0" rpy="0 0 0"/>
+      <inertia ixx="0.0001" iyy="0.0001" izz="0.0001" ixy="0" ixz="0" iyz="0"/>
+    </inertial>
     <visual>
       <geometry>
@@ -100,4 +120,9 @@
   </link>
   <link name="joint6">
+    <inertial>
+      <mass value="0.001"/>
+      <origin xyz="0 0 0" rpy="0 0 0"/>
+      <inertia ixx="0.0001" iyy="0.0001" izz="0.0001" ixy="0" ixz="0" iyz="0"/>
+    </inertial>
     <visual>
       <geometry>
@@ -116,4 +141,9 @@
   </link>
   <link name="joint6_flange">
+    <inertial>
+      <mass value="0.001"/>
+      <origin xyz="0 0 0" rpy="0 0 0"/>
+      <inertia ixx="0.0001" iyy="0.0001" izz="0.0001" ixy="0" ixz="0" iyz="0"/>
+    </inertial>
     <visual>
       <geometry>
