Commit message: Fixed .jpg mesh import

File: ur5_cell/src/ur5_cell_motus/urdf/ur5_cell.urdf.xacro (robot description, xacro)
@@ -3,4 +3,6 @@
   <xacro:arg name="controllers_yaml_path" default=""/>
   <xacro:arg name="namespace" default=""/>
+  <xacro:arg name="home_pose" default=""/>
+  <xacro:property name="_motus_home_pose" value="$(arg home_pose)"/>
    <!-- robot name parameter -->
    <xacro:arg name="name" default="ur"/>
@@ -46,30 +48,42 @@
       <joint name="shoulder_pan_joint">
         <command_interface name="position"/>
-        <state_interface name="position"/>
+        <state_interface name="position">
+          <param name="initial_value">${float(str(_motus_home_pose).split(',')[0]) if str(_motus_home_pose).strip() and len(str(_motus_home_pose).split(',')) > 0 else 0.0}</param>
+        </state_interface>
         <state_interface name="velocity"/>
       </joint>
       <joint name="shoulder_lift_joint">
         <command_interface name="position"/>
-        <state_interface name="position"/>
+        <state_interface name="position">
+          <param name="initial_value">${float(str(_motus_home_pose).split(',')[1]) if str(_motus_home_pose).strip() and len(str(_motus_home_pose).split(',')) > 1 else 0.0}</param>
+        </state_interface>
         <state_interface name="velocity"/>
       </joint>
       <joint name="elbow_joint">
         <command_interface name="position"/>
-        <state_interface name="position"/>
+        <state_interface name="position">
+          <param name="initial_value">${float(str(_motus_home_pose).split(',')[2]) if str(_motus_home_pose).strip() and len(str(_motus_home_pose).split(',')) > 2 else 0.0}</param>
+        </state_interface>
         <state_interface name="velocity"/>
       </joint>
       <joint name="wrist_1_joint">
         <command_interface name="position"/>
-        <state_interface name="position"/>
+        <state_interface name="position">
+          <param name="initial_value">${float(str(_motus_home_pose).split(',')[3]) if str(_motus_home_pose).strip() and len(str(_motus_home_pose).split(',')) > 3 else 0.0}</param>
+        </state_interface>
         <state_interface name="velocity"/>
       </joint>
       <joint name="wrist_2_joint">
         <command_interface name="position"/>
-        <state_interface name="position"/>
+        <state_interface name="position">
+          <param name="initial_value">${float(str(_motus_home_pose).split(',')[4]) if str(_motus_home_pose).strip() and len(str(_motus_home_pose).split(',')) > 4 else 0.0}</param>
+        </state_interface>
         <state_interface name="velocity"/>
       </joint>
       <joint name="wrist_3_joint">
         <command_interface name="position"/>
-        <state_interface name="position"/>
+        <state_interface name="position">
+          <param name="initial_value">${float(str(_motus_home_pose).split(',')[5]) if str(_motus_home_pose).strip() and len(str(_motus_home_pose).split(',')) > 5 else 0.0}</param>
+        </state_interface>
         <state_interface name="velocity"/>
       </joint>

File: ur8long_cell/src/ur8long_cell_motus/urdf/ur8long_cell.urdf.xacro (robot description, xacro)
@@ -42,5 +42,5 @@
      <origin xyz="0 0 0" rpy="0 0 0" />          <!-- position robot in the world -->
    </xacro:ur_robot>
-  <ros2_control name="ur3_cell_motus_GazeboSystem" type="system">
+  <ros2_control name="ur8long_cell_motus_GazeboSystem" type="system">
     <hardware>
       <plugin>gz_ros2_control/GazeboSimSystem</plugin>
